Commit message: Update GO2 SLAM, Nav2, RTABMap, EKF and mapping configurations

File: src/unitree_go2_ros2/unitree_go2_description/urdf/lidar_4D_lidar.xacro (robot description, xacro)
@@ -31,5 +31,5 @@
         <child link="lidar_l1_link"/>
         <!-- <origin rpy="2.94 0 1.5705" xyz="0.25 -0.038 -0.03"/> -->
-        <origin rpy="2.879 0.0 1.5705" xyz="0.25 -0.038 -0.03"/>
+        <origin rpy="0 0 0" xyz="0.25 0.0 0.12"/>
     </joint>
     <gazebo reference="lidar_l1_link">
@@ -67,4 +67,38 @@
             <always_on>1</always_on>
         </sensor>
+        <sensor name="scan_2d" type="gpu_lidar">
+            <topic>scan</topic>
+            <update_rate>10</update_rate>
+            <gz_frame_id>lidar_l1_link</gz_frame_id>
+            <lidar>
+                <scan>
+                    <horizontal>
+                        <samples>720</samples>
+                        <resolution>1</resolution>
+                        <min_angle>-3.14159</min_angle>
+                        <max_angle>3.14159</max_angle>
+                    </horizontal>
+                    <vertical>
+                        <samples>1</samples>
+                        <resolution>1</resolution>
+                        <min_angle>0.0</min_angle>
+                        <max_angle>0.0</max_angle>
+                    </vertical>
+                </scan>
+                <range>
+                    <min>0.2</min>
+                    <max>20.0</max>
+                    <resolution>0.01</resolution>
+                </range>
+                <noise>
+                    <type>gaussian</type>
+                    <mean>0.0</mean>
+                    <stddev>0.005</stddev>
+                </noise>
+                <frame_id>lidar_l1_link</frame_id>
+            </lidar>
+            <visualize>true</visualize>
+            <always_on>1</always_on>
+        </sensor>
     </gazebo>
 </robot>

File: src/unitree_go2_ros2/unitree_go2_description/urdf/velodyne.xacro (robot description, xacro)
@@ -84,3 +84,38 @@
         </sensor>
     </gazebo>
+    <gazebo reference="velodyne">
+  <sensor name="slam_2d_lidar" type="ray">
+    <topic>scan</topic>
+    <update_rate>10</update_rate>
+    <gz_frame_id>velodyne</gz_frame_id>
+    <ray>
+      <scan>
+        <horizontal>
+          <samples>720</samples>
+          <resolution>1</resolution>
+          <min_angle>-3.14159</min_angle>
+          <max_angle>3.14159</max_angle>
+        </horizontal>
+        <vertical>
+          <samples>1</samples>
+          <resolution>1</resolution>
+          <min_angle>0.0</min_angle>
+          <max_angle>0.0</max_angle>
+        </vertical>
+      </scan>
+      <range>
+        <min>0.2</min>
+        <max>20.0</max>
+        <resolution>0.01</resolution>
+      </range>
+      <noise>
+        <type>gaussian</type>
+        <mean>0.0</mean>
+        <stddev>0.005</stddev>
+      </noise>
+    </ray>
+    <always_on>1</always_on>
+    <visualize>true</visualize>
+  </sensor>
+</gazebo>
 </robot>
